File: 4CPCB/4CPCB.kicad_sch (KiCad schematic)
At the start: 0 parts

Commit message: pre-STM32 signal routing
Other:
- removed sheet drh
- removed sheet drh1
- removed sheet drh3
Changed lines of the file:
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@@
 	(paper "A4")
-	(sheet
-		(at 18.034 50.8)
-		(size 49.276 33.02)
-		(exclude_from_sim no)
-		(in_bom yes)
-		(on_board yes)
-		(dnp no)
-		(fields_autoplaced yes)
-		(stroke
-			(width 0.1524)
-			(type solid)
-		)
-		(fill
-			(color 0 0 0 0.0000)
-		)
-		(property "Sheetname" "drh"
-			(at 18.034 50.0884 0)
-			(effects
-				(font
-					(size 1.27 1.27)
-				)
-				(justify left bottom)
-			)
-		)
-		(property "Sheetfile" "drh.kicad_sch"
-			(at 18.034 84.4046 0)
-			(effects
-				(font
-					(size 1.27 1.27)
-				)
-				(justify left top)
-			)
-		)
-		(instances
-			(project "4CPCB"
-				(path "/0f9f1327-d1b6-4021-a070-292f84c5eae1"
-					(page "2")
-				)
-			)
-		)
-	)
 	(sheet
 		(at 83.82 49.53)
@@
 				)
 			)
-		)
-	)
-	(sheet
-		(at 19.05 96.52)
-		(size 49.276 33.02)
-		(exclude_from_sim no)
-		(in_bom yes)
-		(on_board yes)
-		(dnp no)
-		(fields_autoplaced yes)
-		(stroke
-			(width 0.1524)
-			(type solid)
-		)
-		(fill
-			(color 0 0 0 0.0000)
-		)
-		(property "Sheetname" "drh1"
-			(at 19.05 95.8084 0)
-			(effects
-				(font
-					(size 1.27 1.27)
-				)
-				(justify left bottom)
-			)
-		)
-		(property "Sheetfile" "drh.kicad_sch"
-			(at 19.05 130.1246 0)
-			(effects
-				(font
-					(size 1.27 1.27)
-				)
-				(justify left top)
-			)
-		)
-		(instances
-			(project "4CPCB"
-				(path "/0f9f1327-d1b6-4021-a070-292f84c5eae1"
-					(page "3")
-				)
-			)
-		)
-	)
-	(sheet
-		(at 82.55 93.98)
-		(size 49.276 33.02)
-		(exclude_from_sim no)
-		(in_bom yes)
-		(on_board yes)
-		(dnp no)
-		(fields_autoplaced yes)
-		(stroke
-			(width 0.1524)
-			(type solid)
-		)
-		(fill
-			(color 0 0 0 0.0000)
-		)
-		(property "Sheetname" "drh3"
-			(at 82.55 93.2684 0)
-			(effects
-				(font
-					(size 1.27 1.27)
-				)
-				(justify left bottom)
-			)
-		)
-		(property "Sheetfile" "drh.kicad_sch"
-			(at 82.55 127.5846 0)
-			(effects
-				(font
-					(size 1.27 1.27)
-				)
-				(justify left top)
-			)
-		)
-		(instances
-			(project "4CPCB"
-				(path "/0f9f1327-d1b6-4021-a070-292f84c5eae1"
-					(page "5")
-				)
-			)
