File: 4CPCB/pcb/drh.kicad_sch (KiCad schematic)
At the start: 50 parts, among them Q10 ${PARTNUMBER}, Q11 ${PARTNUMBER}, Q12 ${PARTNUMBER}, Q9 ${PARTNUMBER}, U3 ${PARTNUMBER}

Commit message: pre-STM32 signal routing
Parts:
- removed C40, C41, C43: ${PARTNUMBER}, 0603L, symbol Capacitor_Ceramic:root_1_C1608X7R1H103K_Capacitor_Ceramic.IntLib
- removed NT11: Net-Tie, Net-Tie_10mil, symbol MiscParts:root_0_Net-Tie_MiscParts.IntLib
- removed R27: ${PARTNUMBER}, 0603L, symbol Resistor_0603:root_1_CRCW06030000Z0EA_Resistor_0603.IntLib
- removed TP34, TP37, TP39, TP42: ${PARTNUMBER}, Keystone5007, symbol Connectors:root_0_5007_Connectors.IntLib
- added C10, C11, C13: ${PARTNUMBER}, Capacitor_SMD:C_0603_1608Metric_Pad1.08x0.95mm_HandSolder, symbol Capacitor_Ceramic:root_1_C1608X7R1H103K_Capacitor_Ceramic.IntLib
- added J10: Conn_01x02, Connector_JST:JST_VH_B2P-VH_1x02_P3.96mm_Vertical, symbol Connector_Generic:Conn_01x02
- added NT3: Net-Tie, NetTie:NetTie-2_SMD_Pad0.5mm, symbol MiscParts:root_2_Net-Tie_MiscParts.IntLib
- added R6: ${PARTNUMBER}, Resistor_SMD:R_0603_1608Metric_Pad0.98x0.95mm_HandSolder, symbol Resistor_0603:root_1_CRCW06030000Z0EA_Resistor_0603.IntLib
- added TP11, TP14, TP6, TP9: AVDD, TestPoint:TestPoint_Pad_D1.5mm, symbol MiscParts:root_0_TESTPOINT_MiscParts.IntLib
- C1: renamed from C31; footprint 1210L -> Easyeda:C0805
- C12: renamed from C42; footprint 0603L -> Capacitor_SMD:C_0603_1608Metric_Pad1.08x0.95mm_HandSolder; now not fitted
- C2: renamed from C32; footprint 0603L -> Easyeda:C0603
- C6: renamed from C36; footprint 0603L -> Easyeda:C0603
- H1: renamed from H2; LCSC (none) -> C5188489
- NT1: renamed from NT9; footprint Net-Tie_10mil -> NetTie:NetTie-2_SMD_Pad0.5mm
- NT2: renamed from NT10; footprint Net-Tie_10mil -> NetTie:NetTie-2_SMD_Pad0.5mm
- NT4: renamed from NT12; footprint Net-Tie_10mil -> NetTie:NetTie-2_SMD_Pad0.5mm
- R5: renamed from R26; footprint 0603L -> Resistor_SMD:R_0603_1608Metric_Pad0.98x0.95mm_HandSolder; now not fitted
- renumbered C44 to C14, C45 to C15, C33 to C3, C34 to C4, C35 to C5, C37 to C7, C38 to C8, C39 to C9, Q9 to Q1, Q10 to Q2, Q11 to Q3, Q12 to Q4, R22 to R1, R32 to R10, R33 to R11, R23 to R2, R24 to R3, R25 to R4, R28 to R7, R29 to R8, R31 to R9, TP29 to TP1, TP38 to TP10, TP40 to TP12, TP41 to TP13, TP30 to TP2, TP31 to TP3, TP32 to TP4, TP33 to TP5, TP35 to TP7, TP36 to TP8, U3 to U1
Connections:
- net GND: now also NT3.1, R6.1, TP11.1
- net OUT1: now also C13.1, J10.1 (Pin_1)
- net OUT2: now also C10.2, C11.1, J10.2 (Pin_2)
- net S_N: now also NT3.2
- net VM: now also C10.1
- net VREF: now also R6.2
- net at NT2.1, Q2.1 (S), Q2.2 (S)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: now also C11.2, C13.2, TP9.1
- net at Q2.4 (G), R8.1: now also TP6.1
- net at Q4.4 (G), R11.2: now also TP14.1
Other:
- moved on the sheet: C1, C14, C15, C2, C3, C4, C5, C6, C7, C8, C9, H1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
