File: 4CPCB/pcb/drh.kicad_sch (KiCad schematic)
At the start: 51 parts, among them J10 Conn_01x02, Q1 ${PARTNUMBER}, Q2 ${PARTNUMBER}, Q3 ${PARTNUMBER}, Q4 ${PARTNUMBER}, U1 ${PARTNUMBER}

Commit message: Add project-local KiCad libraries
Parts:
- R5, R6: now left out of the parts list
Connections:
- net 3.3V renamed +3.3V
