File: 4CPCB/pcb/pcb.kicad_pcb (KiCad board)
At the start: 2 copper layers, 50 parts, among them Q1 CSD18532Q5B, Q2 CSD18532Q5B, Q3 CSD18532Q5B, Q4 CSD18532Q5B, U1 DRV8701ERGER

Commit message: checkpoints
Parts:
- removed C10, C11, C12, C13: DNP, Capacitor_SMD:C_0603_1608Metric_Pad1.08x0.95mm_HandSolder
- removed H1: 691 101 710 002, Easyeda:CONN-TH_MX635-6.35-02P-GN01-CU-PS-A
- added C16: GRM32ER71H106KA12L, Easyeda:C0805, F.Cu at (296.0, 284.6)
- added C17: C1608X7R1H104K, Easyeda:C0402, F.Cu at (287.5, 290.7)
- added C18: GRM188R70J105KA01D, Easyeda:C0603, F.Cu at (295.4, 273.8)
- added C19: GRM188R70J105KA01D, Easyeda:C0603, F.Cu at (295.4, 276.4)
- added C20: C1608X7R1C105K, Easyeda:C0402, F.Cu at (287.5, 292.9)
- added C21: C1608X7R1H104K, Easyeda:C0402, F.Cu at (287.5, 295.0)
- added C22: GRM188R70J105KA01D, Easyeda:C0603, F.Cu at (295.4, 279.1)
- added C23: ECA-1HM471, Easyeda:CAP-TH_BD10.0-P5.00-D0.6-FD, F.Cu at (269.8, 278.1)
- added C24: GRM155R71C102KA01D, Easyeda:C0402, F.Cu at (287.5, 297.1)
- added C25: DNP, Capacitor_SMD:C_0603_1608Metric_Pad1.08x0.95mm_HandSolder, F.Cu at (291.3, 273.7)
- added C26: DNP, Capacitor_SMD:C_0603_1608Metric_Pad1.08x0.95mm_HandSolder, F.Cu at (291.3, 276.2)
- added C27: DNP, Capacitor_SMD:C_0603_1608Metric_Pad1.08x0.95mm_HandSolder, F.Cu at (291.3, 278.7)
- added C28: DNP, Capacitor_SMD:C_0603_1608Metric_Pad1.08x0.95mm_HandSolder, F.Cu at (291.3, 281.2)
- added C29: GRM188R70J105KA01D, Easyeda:C0603, F.Cu at (295.4, 281.8)
- added C30: ECA-1HM471, Easyeda:CAP-TH_BD10.0-P5.00-D0.6-FD, F.Cu at (269.8, 289.3)
- added C31: GRM32ER71H106KA12L, Easyeda:C0805, F.Cu at (296.0, 320.6)
- added C32: C1608X7R1H104K, Easyeda:C0402, F.Cu at (287.5, 326.7)
- added C33: GRM188R70J105KA01D, Easyeda:C0603, F.Cu at (295.4, 309.7)
- added C34: GRM188R70J105KA01D, Easyeda:C0603, F.Cu at (295.4, 312.4)
- added C35: C1608X7R1C105K, Easyeda:C0402, F.Cu at (287.5, 328.8)
- added C36: C1608X7R1H104K, Easyeda:C0402, F.Cu at (287.5, 331.0)
- added C37: GRM188R70J105KA01D, Easyeda:C0603, F.Cu at (295.4, 315.1)
- added C38: ECA-1HM471, Easyeda:CAP-TH_BD10.0-P5.00-D0.6-FD, F.Cu at (269.8, 314.0)
- added C39: GRM155R71C102KA01D, Easyeda:C0402, F.Cu at (287.5, 333.1)
- added C40: DNP, Capacitor_SMD:C_0603_1608Metric_Pad1.08x0.95mm_HandSolder, F.Cu at (291.3, 309.7)
- added C41: DNP, Capacitor_SMD:C_0603_1608Metric_Pad1.08x0.95mm_HandSolder, F.Cu at (291.3, 312.2)
- added C42: DNP, Capacitor_SMD:C_0603_1608Metric_Pad1.08x0.95mm_HandSolder, F.Cu at (291.3, 314.7)
- added C43: DNP, Capacitor_SMD:C_0603_1608Metric_Pad1.08x0.95mm_HandSolder, F.Cu at (291.3, 317.2)
- added C44: GRM188R70J105KA01D, Easyeda:C0603, F.Cu at (295.4, 317.8)
- added C45: ECA-1HM471, Easyeda:CAP-TH_BD10.0-P5.00-D0.6-FD, F.Cu at (269.8, 325.3)
- added C46: GRM32ER71H106KA12L, Easyeda:C0805, F.Cu at (345.2, 235.8)
- added C47: C1608X7R1H104K, Easyeda:C0402, F.Cu at (336.8, 241.9)
- added C48: GRM188R70J105KA01D, Easyeda:C0603, F.Cu at (344.7, 225.0)
- added C49: GRM188R70J105KA01D, Easyeda:C0603, F.Cu at (344.7, 227.6)
- added C50: C1608X7R1C105K, Easyeda:C0402, F.Cu at (336.8, 244.1)
- added C51: C1608X7R1H104K, Easyeda:C0402, F.Cu at (336.8, 246.2)
- added C52: GRM188R70J105KA01D, Easyeda:C0603, F.Cu at (344.7, 230.3)
- added C53: ECA-1HM471, Easyeda:CAP-TH_BD10.0-P5.00-D0.6-FD, F.Cu at (319.1, 229.2)
- added C54: GRM155R71C102KA01D, Easyeda:C0402, F.Cu at (336.8, 248.3)
- added C55: DNP, Capacitor_SMD:C_0603_1608Metric_Pad1.08x0.95mm_HandSolder, F.Cu at (340.5, 224.9)
- added C56: DNP, Capacitor_SMD:C_0603_1608Metric_Pad1.08x0.95mm_HandSolder, F.Cu at (340.5, 227.4)
- added C57: DNP, Capacitor_SMD:C_0603_1608Metric_Pad1.08x0.95mm_HandSolder, F.Cu at (340.5, 229.9)
- added C58: DNP, Capacitor_SMD:C_0603_1608Metric_Pad1.08x0.95mm_HandSolder, F.Cu at (340.5, 232.4)
- added C59: GRM188R70J105KA01D, Easyeda:C0603, F.Cu at (344.7, 233.0)
- added C60: ECA-1HM471, Easyeda:CAP-TH_BD10.0-P5.00-D0.6-FD, F.Cu at (319.1, 240.5)
- added C61: GRM188R70J105KA01D, Easyeda:C0402, F.Cu at (120.1, 71.8)
- added C62: C1608X7R1H104K, Easyeda:C0402, F.Cu at (120.1, 73.9)
- added C63: GRM188R70J105KA01D, Easyeda:C0402, F.Cu at (120.1, 76.1)
- added C64: C1608X7R1H104K, Easyeda:C0402, F.Cu at (120.1, 78.2)
- added C65: GRM32ER71H106KA12L, Easyeda:C0402, F.Cu at (123.0, 71.8)
- added C66: C1608X7R1H104K, Easyeda:C0402, F.Cu at (123.0, 73.9)
- added C67: C1608X7R1H104K, Easyeda:C0402, F.Cu at (123.0, 76.1)
- added C68: C1608X7R1H104K, Easyeda:C0402, F.Cu at (123.0, 78.2)
- added C69: C1608X7R1H104K, Easyeda:C0402, F.Cu at (125.9, 71.8)
- added C70: 10uF, Easyeda:C0805, F.Cu at (256.0, 37.0)
- added C71: 22uF, Easyeda:C0805, F.Cu at (246.0, 29.0)
- added C72: C1608X7R1H104K, Easyeda:C0402, F.Cu at (125.9, 73.9)
- added C73: C1608X7R1H104K, Easyeda:C0402, F.Cu at (125.9, 76.1)
- added J1: Conn_01x04, Connector_PinSocket_2.54mm:PinSocket_1x04_P2.54mm_Vertical, F.Cu at (126.1, 41.8)
- added J10: Conn_01x02, Connector_JST:JST_VH_B2P-VH_1x02_P3.96mm_Vertical, F.Cu at (17.7, 266.1)
- added J11: Conn_01x02, Connector_JST:JST_VH_B2P-VH_1x02_P3.96mm_Vertical, F.Cu at (292.5, 292.2)
- added J12: Conn_01x02, Connector_JST:JST_VH_B2P-VH_1x02_P3.96mm_Vertical, F.Cu at (292.5, 328.2)
- added J13: Conn_01x02, Connector_JST:JST_VH_B2P-VH_1x02_P3.96mm_Vertical, F.Cu at (341.8, 243.4)
- added J18: Conn_01x04, Connector_JST:JST_XH_B4B-XH-A_1x04_P2.50mm_Vertical, F.Cu at (112.8, 42.9)
- added J19: Conn_01x04, Connector_JST:JST_XH_B4B-XH-A_1x04_P2.50mm_Vertical, F.Cu at (112.8, 50.7)
- added J2: XT90PW-F, Easyeda:AMASS_XT90PW-F, F.Cu at (96.5, 51.9)
- added J20: Conn_01x04, Connector_JST:JST_XH_B4B-XH-A_1x04_P2.50mm_Vertical, F.Cu at (112.8, 58.5)
- added J21: Conn_01x04, Connector_JST:JST_XH_B4B-XH-A_1x04_P2.50mm_Vertical, F.Cu at (112.8, 66.3)
- added J22: Conn_01x03, Connector_PinHeader_2.54mm:PinHeader_1x03_P2.54mm_Vertical, F.Cu at (126.1, 54.0)
- added L1: GZ1608D601TF, Easyeda:L0603, F.Cu at (125.8, 62.6)
- added NT10: Net-Tie, NetTie:NetTie-2_SMD_Pad0.5mm, F.Cu at (297.4, 302.5)
- added NT11: Net-Tie, NetTie:NetTie-2_SMD_Pad0.5mm, F.Cu at (297.4, 304.0)
- added NT12: Net-Tie, NetTie:NetTie-2_SMD_Pad0.5mm, F.Cu at (297.4, 305.5)
- added NT13: Net-Tie, NetTie:NetTie-2_SMD_Pad0.5mm, F.Cu at (346.7, 216.2)
- added NT14: Net-Tie, NetTie:NetTie-2_SMD_Pad0.5mm, F.Cu at (346.7, 217.7)
- added NT15: Net-Tie, NetTie:NetTie-2_SMD_Pad0.5mm, F.Cu at (346.7, 219.2)
- added NT16: Net-Tie, NetTie:NetTie-2_SMD_Pad0.5mm, F.Cu at (346.7, 220.7)
- added NT5: Net-Tie, NetTie:NetTie-2_SMD_Pad0.5mm, F.Cu at (297.4, 265.0)
- added NT6: Net-Tie, NetTie:NetTie-2_SMD_Pad0.5mm, F.Cu at (297.4, 266.5)
- added NT7: Net-Tie, NetTie:NetTie-2_SMD_Pad0.5mm, F.Cu at (297.4, 268.0)
- added NT8: Net-Tie, NetTie:NetTie-2_SMD_Pad0.5mm, F.Cu at (297.4, 269.5)
- added NT9: Net-Tie, NetTie:NetTie-2_SMD_Pad0.5mm, F.Cu at (297.4, 301.0)
- added Q10: CSD18532Q5B, Easyeda:VSON-CLIP-8_L5.0-W6.0-P1.27-BL, F.Cu at (274.1, 304.2)
- added Q11: CSD18532Q5B, Easyeda:VSON-CLIP-8_L5.0-W6.0-P1.27-BL, F.Cu at (280.7, 304.2)
- added Q12: CSD18532Q5B, Easyeda:VSON-CLIP-8_L5.0-W6.0-P1.27-BL, F.Cu at (287.3, 304.2)
- added Q13: CSD18532Q5B, Easyeda:VSON-CLIP-8_L5.0-W6.0-P1.27-BL, F.Cu at (316.8, 219.4)
- added Q14: CSD18532Q5B, Easyeda:VSON-CLIP-8_L5.0-W6.0-P1.27-BL, F.Cu at (323.4, 219.4)
- added Q15: CSD18532Q5B, Easyeda:VSON-CLIP-8_L5.0-W6.0-P1.27-BL, F.Cu at (330.0, 219.4)
- added Q16: CSD18532Q5B, Easyeda:VSON-CLIP-8_L5.0-W6.0-P1.27-BL, F.Cu at (336.6, 219.4)
- added Q5: CSD18532Q5B, Easyeda:VSON-CLIP-8_L5.0-W6.0-P1.27-BL, F.Cu at (267.5, 268.2)
- added Q6: CSD18532Q5B, Easyeda:VSON-CLIP-8_L5.0-W6.0-P1.27-BL, F.Cu at (274.1, 268.2)
- added Q7: CSD18532Q5B, Easyeda:VSON-CLIP-8_L5.0-W6.0-P1.27-BL, F.Cu at (280.7, 268.2)
- added Q8: CSD18532Q5B, Easyeda:VSON-CLIP-8_L5.0-W6.0-P1.27-BL, F.Cu at (287.3, 268.2)
- added Q9: CSD18532Q5B, Easyeda:VSON-CLIP-8_L5.0-W6.0-P1.27-BL, F.Cu at (267.5, 304.2)
- added R12: CRCW060310K0JNEA, Easyeda:R0402, F.Cu at (287.6, 273.5)
- added R13: CRCW060310K0JNEA, Easyeda:R0402, F.Cu at (287.6, 275.6)
- added R14: CRCW06037K50JNEA, Easyeda:R0402, F.Cu at (287.6, 277.8)
- added R15: CRCW060310K0JNEA, Easyeda:R0402, F.Cu at (287.6, 279.9)
- added R16: DNP, Resistor_SMD:R_0603_1608Metric_Pad0.98x0.95mm_HandSolder, F.Cu at (291.3, 283.7)
- added R17: DNP, Resistor_SMD:R_0603_1608Metric_Pad0.98x0.95mm_HandSolder, F.Cu at (291.3, 286.2)
- added R18: CRCW06030000Z0EA, Easyeda:R0402, F.Cu at (287.6, 282.1)
- added R19: CRCW06030000Z0EA, Easyeda:R0402, F.Cu at (287.6, 284.2)
- added R20: CRA2512-FZ-R010ELF, Easyeda:R2818, F.Cu at (280.0, 293.5)
- added R21: CRCW06030000Z0EA, Easyeda:R0402, F.Cu at (287.6, 286.4)
- added R22: CRCW06030000Z0EA, Easyeda:R0402, F.Cu at (287.6, 288.6)
- added R23: CRCW060310K0JNEA, Easyeda:R0402, F.Cu at (287.6, 309.5)
- added R24: CRCW060310K0JNEA, Easyeda:R0402, F.Cu at (287.6, 311.6)
- added R25: CRCW06037K50JNEA, Easyeda:R0402, F.Cu at (287.6, 313.8)
- added R26: CRCW060310K0JNEA, Easyeda:R0402, F.Cu at (287.6, 315.9)
- added R27: DNP, Resistor_SMD:R_0603_1608Metric_Pad0.98x0.95mm_HandSolder, F.Cu at (291.3, 319.7)
- added R28: DNP, Resistor_SMD:R_0603_1608Metric_Pad0.98x0.95mm_HandSolder, F.Cu at (291.3, 322.2)
- added R29: CRCW06030000Z0EA, Easyeda:R0402, F.Cu at (287.6, 318.1)
- added R30: CRCW06030000Z0EA, Easyeda:R0402, F.Cu at (287.6, 320.2)
- added R31: CRA2512-FZ-R010ELF, Easyeda:R2818, F.Cu at (280.0, 329.5)
- added R32: CRCW06030000Z0EA, Easyeda:R0402, F.Cu at (287.6, 322.4)
- added R33: CRCW06030000Z0EA, Easyeda:R0402, F.Cu at (287.6, 324.5)
- added R34: CRCW060310K0JNEA, Easyeda:R0402, F.Cu at (336.8, 224.7)
- added R35: CRCW060310K0JNEA, Easyeda:R0402, F.Cu at (336.8, 226.8)
- added R36: CRCW06037K50JNEA, Easyeda:R0402, F.Cu at (336.8, 229.0)
- added R37: CRCW060310K0JNEA, Easyeda:R0402, F.Cu at (336.8, 231.2)
- added R38: DNP, Resistor_SMD:R_0603_1608Metric_Pad0.98x0.95mm_HandSolder, F.Cu at (340.5, 234.9)
- added R39: DNP, Resistor_SMD:R_0603_1608Metric_Pad0.98x0.95mm_HandSolder, F.Cu at (340.5, 237.4)
- added R40: CRCW06030000Z0EA, Easyeda:R0402, F.Cu at (336.8, 233.3)
- added R41: CRCW06030000Z0EA, Easyeda:R0402, F.Cu at (336.8, 235.4)
- added R42: CRA2512-FZ-R010ELF, Easyeda:R2818, F.Cu at (329.3, 244.7)
- added R43: CRCW06030000Z0EA, Easyeda:R0402, F.Cu at (336.8, 237.6)
- added R44: CRCW06030000Z0EA, Easyeda:R0402, F.Cu at (336.8, 239.8)
- added R45: CRCW06030000Z0EA, Easyeda:R0402, F.Cu at (260.5, 37.1)
- added R46: CRCW06030000Z0EA, Easyeda:R0402, F.Cu at (263.5, 37.0)
- added TP15: VM, TestPoint:TestPoint_Pad_D1.5mm, F.Cu at (277.2, 274.2)
- added TP16: VM, TestPoint:TestPoint_Pad_D1.5mm, F.Cu at (277.2, 277.8)
- added TP17: AVDD, TestPoint:TestPoint_Pad_D1.5mm, F.Cu at (277.2, 281.3)
- added TP18: AVDD, TestPoint:TestPoint_Pad_D1.5mm, F.Cu at (277.2, 284.9)
- added TP19: AVDD, TestPoint:TestPoint_Pad_D1.5mm, F.Cu at (277.2, 288.4)
- added TP20: AVDD, TestPoint:TestPoint_Pad_D1.5mm, F.Cu at (280.7, 274.2)
- added TP21: AVDD, TestPoint:TestPoint_Pad_D1.5mm, F.Cu at (280.7, 277.8)
- added TP22: AVDD, TestPoint:TestPoint_Pad_D1.5mm, F.Cu at (280.7, 281.3)
- added TP23: AVDD, TestPoint:TestPoint_Pad_D1.5mm, F.Cu at (280.7, 284.9)
- added TP24: AVDD, TestPoint:TestPoint_Pad_D1.5mm, F.Cu at (280.7, 288.4)
- added TP25: AVDD, TestPoint:TestPoint_Pad_D1.5mm, F.Cu at (284.3, 274.2)
- added TP26: AVDD, TestPoint:TestPoint_Pad_D1.5mm, F.Cu at (284.3, 277.8)
- added TP27: AVDD, TestPoint:TestPoint_Pad_D1.5mm, F.Cu at (284.3, 281.3)
- added TP28: AVDD, TestPoint:TestPoint_Pad_D1.5mm, F.Cu at (284.3, 284.9)
- added TP29: VM, TestPoint:TestPoint_Pad_D1.5mm, F.Cu at (277.2, 310.2)
- added TP30: VM, TestPoint:TestPoint_Pad_D1.5mm, F.Cu at (277.2, 313.7)
- added TP31: AVDD, TestPoint:TestPoint_Pad_D1.5mm, F.Cu at (277.2, 317.3)
- added TP32: AVDD, TestPoint:TestPoint_Pad_D1.5mm, F.Cu at (277.2, 320.8)
- added TP33: AVDD, TestPoint:TestPoint_Pad_D1.5mm, F.Cu at (277.2, 324.4)
- added TP34: AVDD, TestPoint:TestPoint_Pad_D1.5mm, F.Cu at (280.7, 310.2)
- added TP35: AVDD, TestPoint:TestPoint_Pad_D1.5mm, F.Cu at (280.7, 313.7)
- added TP36: AVDD, TestPoint:TestPoint_Pad_D1.5mm, F.Cu at (280.7, 317.3)
- added TP37: AVDD, TestPoint:TestPoint_Pad_D1.5mm, F.Cu at (280.7, 320.8)
- added TP38: AVDD, TestPoint:TestPoint_Pad_D1.5mm, F.Cu at (280.7, 324.4)
- added TP39: AVDD, TestPoint:TestPoint_Pad_D1.5mm, F.Cu at (284.3, 310.2)
- added TP40: AVDD, TestPoint:TestPoint_Pad_D1.5mm, F.Cu at (284.3, 313.7)
- added TP41: AVDD, TestPoint:TestPoint_Pad_D1.5mm, F.Cu at (284.3, 317.3)
- added TP42: AVDD, TestPoint:TestPoint_Pad_D1.5mm, F.Cu at (284.3, 320.8)
- added TP43: VM, TestPoint:TestPoint_Pad_D1.5mm, F.Cu at (326.4, 225.4)
- added TP44: VM, TestPoint:TestPoint_Pad_D1.5mm, F.Cu at (326.4, 228.9)
- added TP45: AVDD, TestPoint:TestPoint_Pad_D1.5mm, F.Cu at (326.4, 232.5)
- added TP46: AVDD, TestPoint:TestPoint_Pad_D1.5mm, F.Cu at (326.4, 236.1)
- added TP47: AVDD, TestPoint:TestPoint_Pad_D1.5mm, F.Cu at (326.4, 239.6)
- added TP48: AVDD, TestPoint:TestPoint_Pad_D1.5mm, F.Cu at (330.0, 225.4)
- added TP49: AVDD, TestPoint:TestPoint_Pad_D1.5mm, F.Cu at (330.0, 228.9)
- added TP50: AVDD, TestPoint:TestPoint_Pad_D1.5mm, F.Cu at (330.0, 232.5)
- added TP51: AVDD, TestPoint:TestPoint_Pad_D1.5mm, F.Cu at (330.0, 236.1)
- added TP52: AVDD, TestPoint:TestPoint_Pad_D1.5mm, F.Cu at (330.0, 239.6)
- added TP53: AVDD, TestPoint:TestPoint_Pad_D1.5mm, F.Cu at (333.6, 225.4)
- added TP54: AVDD, TestPoint:TestPoint_Pad_D1.5mm, F.Cu at (333.6, 228.9)
- added TP55: AVDD, TestPoint:TestPoint_Pad_D1.5mm, F.Cu at (333.6, 232.5)
- added TP56: AVDD, TestPoint:TestPoint_Pad_D1.5mm, F.Cu at (333.6, 236.1)
- added U2: DRV8701ERGER, Easyeda:VQFN-24_L4.0-W4.0-P0.50-BL-EP2.5, F.Cu at (293.4, 267.0)
- added U3: DRV8701ERGER, Easyeda:VQFN-24_L4.0-W4.0-P0.50-BL-EP2.5, F.Cu at (293.4, 303.0)
- added U4: DRV8701ERGER, Easyeda:VQFN-24_L4.0-W4.0-P0.50-BL-EP2.5, F.Cu at (342.6, 218.2)
- added U5: STM32G474RETx, Package_QFP:LQFP-64_10x10mm_P0.5mm, F.Cu at (240.5, 44.5)
- added U6: AMS1117-3.3, Easyeda:SOT-223-3_L6.5-W3.4-P2.30-LS7.0-BR, F.Cu at (252.0, 31.0)
- added USB1: HX TYPE-C 16PIN 3MD 385, Easyeda:TYPE-C-SMD_HX-TYPE-C-16PIN, F.Cu at (262.0, 32.6)
- C14, C3, C4, C7: footprint Easyeda:C0805 -> Easyeda:C0603
- C2, C6: footprint Easyeda:C0603 -> Easyeda:C0402
- C5: footprint Easyeda:C0805 -> Easyeda:C0402
- R1, R2, R4: footprint Easyeda:R0805 -> Easyeda:R0402
- R10, R11, R3, R7, R8: footprint Easyeda:R0603 -> Easyeda:R0402
- moved R10 295.1 mm to (4.50, 349.0), turned to 90 degrees
- moved R11 240.7 mm to (33.8, 301.4)
- moved R5 234.9 mm to (37.5, 296.5)
- moved R6 234.9 mm to (37.5, 299.0)
- moved TP12 234.7 mm to (30.5, 290.6)
- moved TP13 234.7 mm to (30.5, 294.1)
- moved TP2 234.7 mm to (23.4, 290.6)
- moved TP3 234.7 mm to (23.4, 294.1)
- moved TP7 234.7 mm to (26.9, 290.6)
- moved TP8 234.7 mm to (26.9, 294.1)
- moved TP1 234.7 mm to (23.4, 287.0)
- moved TP10 234.7 mm to (26.9, 301.2)
- moved TP11 234.7 mm to (30.5, 287.0)
- moved TP14 234.7 mm to (30.5, 297.6)
- moved TP4 234.7 mm to (23.4, 297.6)
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Connections:
- net /drh/GH1 renamed /drh1/GH1
- net /drh/GH2 renamed /drh1/GH2
- net /drh/GL1 renamed /drh1/GL1
- net /drh/GL2 renamed /drh1/GL2
- net /drh/OUT1 renamed /drh1/OUT2
- net /drh/OUT2 renamed /drh1/OUT1
- net /drh/SH1 renamed /drh1/SH1
- net /drh/SH2 renamed /drh1/SH2
- net /drh/SNSOUT renamed /drh1/SNSOUT
- net /drh/SO renamed /SO_1
- net /drh/S_N renamed /drh1/S_N
- net /drh/S_P renamed /drh1/S_P
- net /drh/VCP renamed /drh1/VCP
- net /drh/VREF renamed /VREF
- net /drh/nFAULT renamed /nFAULT_1
- net Net-(C11-Pad2) renamed /drh1/SHUNT_TOP
- U1 pad 12: /drh/IDRIVE -> GND
- U1 pad 13: /drh/nSLEEP -> /nSLEEP
- U1 pad 14: /drh/EN/IN2 -> /EN_1
- U1 pad 15: /drh/PH/IN1 -> /PH_DIR_1
Routing:
- net VM: track 0.00 -> 12.9 mm
- net /D+: track 0.00 -> 12.5 mm
- net /D-: track 0.00 -> 12.3 mm
- net +5V: track 0.00 -> 10.8 mm
- net /drh1/S_N: track 0.00 -> 9.68 mm
- net +3.3V: track 0.00 -> 9.35 mm
- net Net-(U6-VIN): track 0.00 -> 7.53 mm
- net Net-(U1-SO): track 0.00 -> 4.05 mm
- net /drh1/SNSOUT: track 0.00 -> 3.71 mm
- net /VREF: track 0.00 -> 3.58 mm
- net AVDD: track 0.00 -> 3.48 mm
- net /nFAULT_1: track 0.00 -> 3.22 mm
- net DVDD: track 0.00 -> 2.86 mm
- net Net-(U1-CPL): track 0.00 -> 2.44 mm
- net Net-(U1-CPH): track 0.00 -> 1.95 mm
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- added copper zone on F.Cu, net /drh1/OUT1
- added copper zone on F.Cu, net /drh1/OUT2
- added copper zone on F.Cu, net /drh1/SHUNT_TOP
- added copper zone on F.Cu, net VM
Other:
- board text added: "${REFERENCE}"
- board text added: "CRCW06037K50JNEA"
