File: 4CPCB/pcb/pcb.kicad_pcb (KiCad board)
At the start: 2 copper layers, 222 parts, among them J1 Conn_01x04, J10 Conn_01x02, J11 Conn_01x02, J12 Conn_01x02, J13 Conn_01x02, J18 Conn_01x04, J19 Conn_01x04, J2 XT90PW-F, J20 Conn_01x04, J21 Conn_01x04, J22 Conn_01x03, Q1 CSD18532Q5B, Q10 CSD18532Q5B, Q11 CSD18532Q5B, Q12 CSD18532Q5B, Q13 CSD18532Q5B, Q14 CSD18532Q5B, Q15 CSD18532Q5B, Q16 CSD18532Q5B, Q2 CSD18532Q5B, Q3 CSD18532Q5B, Q4 CSD18532Q5B, Q5 CSD18532Q5B, Q6 CSD18532Q5B, Q7 CSD18532Q5B, Q8 CSD18532Q5B, Q9 CSD18532Q5B, U1 DRV8701ERGER, U2 DRV8701ERGER, U3 DRV8701ERGER, U4 DRV8701ERGER, U5 STM32G474RETx, U6 AMS1117-3.3

Commit message: Add project-local KiCad libraries
Parts:
- removed C25, C26, C27, C28, C40, C41, C42, C43, C55, C56, C57, C58: DNP, Capacitor_SMD:C_0603_1608Metric_Pad1.08x0.95mm_HandSolder
- removed R16, R17, R27, R28, R38, R39, R5, R6: DNP, Resistor_SMD:R_0603_1608Metric_Pad0.98x0.95mm_HandSolder
- removed USB1: HX TYPE-C 16PIN 3MD 385, Easyeda:TYPE-C-SMD_HX-TYPE-C-16PIN
- added J25: USB_C_Receptacle_USB2.0_16P, Connector_USB:USB_C_Receptacle_HRO_TYPE-C-31-M-12, F.Cu at (109.5, 57.0)
- TP1, TP10, TP11, TP13, TP14, TP15, TP16, TP17, TP18, TP19, TP2, TP20, TP21, TP22, TP23, TP24, TP25, TP26, TP27, TP28, TP29, TP3, TP30, TP31, TP32, TP33, TP34, TP35, TP36, TP37, TP38, TP39, TP4, TP40, TP41, TP42, TP43, TP44, TP45, TP46, TP47, TP48, TP49, TP5, TP50, TP51, TP52, TP53, TP54, TP55, TP56, TP6, TP7, TP8, TP9: moved to B.Cu
- moved R10 322.4 mm to (185.6, 82.3)
- moved C39 297.4 mm to (134.7, 78.0), turned to 90 degrees
- moved R31 291.0 mm to (130.2, 80.0), turned to -90 degrees
- moved R30 288.0 mm to (119.2, 86.6), turned to 180 degrees
- moved J12 287.4 mm to (132.5, 89.5), turned to 180 degrees
- moved TP39 281.7 mm to (125.5, 77.6)
- moved R33 280.3 mm to (142.7, 84.6), turned to -90 degrees
- moved TP37 279.9 mm to (135.5, 81.6)
- moved NT11 279.8 mm to (133.2, 77.5)
- moved R32 279.6 mm to (145.7, 81.5), turned to 90 degrees
- moved TP42 279.3 mm to (134.5, 85.1)
- moved C36 279.0 mm to (147.7, 89.6)
- moved C35 278.2 mm to (145.6, 89.6), turned to 180 degrees
- moved R29 277.8 mm to (123.3, 94.1), turned to 180 degrees
- moved TP34 277.4 mm to (120.0, 84.1)
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Connections:
- C18 pad 1: AVDD -> /drh2/AVDD
- C19 pad 2: DVDD -> /drh2/DVDD
- C3 pad 1: AVDD -> /drh1/AVDD
- C33 pad 1: AVDD -> /drh3/AVDD
- C34 pad 2: DVDD -> /drh3/DVDD
- C4 pad 2: DVDD -> /drh1/DVDD
- C48 pad 1: AVDD -> /drh4/AVDD
- C49 pad 2: DVDD -> /drh4/DVDD
- R1 pad 1: 3.3V -> +3.3V
- R12 pad 1: 3.3V -> +3.3V
- R13 pad 1: 3.3V -> +3.3V
- R2 pad 1: 3.3V -> +3.3V
- R23 pad 1: 3.3V -> +3.3V
- R24 pad 1: 3.3V -> +3.3V
- R34 pad 1: 3.3V -> +3.3V
- R35 pad 1: 3.3V -> +3.3V
- TP17 pad 1: AVDD -> /drh2/AVDD
- TP18 pad 1: DVDD -> /drh2/DVDD
- TP3 pad 1: AVDD -> /drh1/AVDD
- TP31 pad 1: AVDD -> /drh3/AVDD
- TP32 pad 1: DVDD -> /drh3/DVDD
- TP4 pad 1: DVDD -> /drh1/DVDD
- TP45 pad 1: AVDD -> /drh4/AVDD
- TP46 pad 1: DVDD -> /drh4/DVDD
- U1 pad 7: AVDD -> /drh1/AVDD
- U1 pad 8: DVDD -> /drh1/DVDD
- U2 pad 7: AVDD -> /drh2/AVDD
- U2 pad 8: DVDD -> /drh2/DVDD
- U3 pad 7: AVDD -> /drh3/AVDD
- U3 pad 8: DVDD -> /drh3/DVDD
- U4 pad 7: AVDD -> /drh4/AVDD
- U4 pad 8: DVDD -> /drh4/DVDD
Routing:
- net +3.3V: track 9.35 -> 395.8 mm, vias 0 -> 14
- net /nSLEEP: track 0.00 -> 363.3 mm, vias 0 -> 5
- net /VREF: track 3.58 -> 288.3 mm, vias 0 -> 6
- net /nFAULT_4: track 0.00 -> 240.8 mm, vias 0 -> 7
- net /EN_4: track 0.00 -> 193.5 mm, vias 0 -> 3
- net /PH_DIR_4: track 0.00 -> 185.7 mm
- net /SO_4: track 0.00 -> 184.0 mm
- net /EN_2: track 0.00 -> 138.2 mm, vias 0 -> 3
- net GND: track 0.00 -> 124.6 mm, vias 0 -> 134
- net /SO_2: track 0.00 -> 112.2 mm, vias 0 -> 2
- net /PH_DIR_2: track 0.00 -> 106.7 mm, vias 0 -> 2
- net /PH_DIR_1: track 0.00 -> 97.8 mm, vias 0 -> 2
- net /nFAULT_1: track 3.22 -> 99.0 mm
- net /ENC_2_B: track 0.00 -> 90.5 mm, vias 0 -> 2
- net /nFAULT_2: track 0.00 -> 87.9 mm, vias 0 -> 2
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- added copper zone on F.Cu, net /drh2/OUT1
- added copper zone on F.Cu, net /drh2/OUT2
- added copper zone on F.Cu, net /drh2/SHUNT_TOP
- added copper zone on F.Cu, net /drh3/OUT1
- added copper zone on F.Cu, net /drh3/OUT2
- added copper zone on F.Cu, net /drh3/SHUNT_TOP
- added copper zone on F.Cu, net /drh4/OUT1
- added copper zone on F.Cu, net /drh4/OUT2
- added copper zone on F.Cu, net /drh4/SHUNT_TOP
- added copper zone on F.Cu, net GND
- added copper zone on In1.Cu, net GND
Other:
- board outline added: 100 x 100 mm
- copper layers 2 -> 4
- board text removed: "${REFERENCE}"
- board text removed: "CRCW06037K50JNEA"
