File: hardware/kicad/drh.kicad_sch (KiCad schematic)
At the start: 51 parts, among them J10 Conn_01x02, Q1 ${PARTNUMBER}, Q2 ${PARTNUMBER}, Q3 ${PARTNUMBER}, Q4 ${PARTNUMBER}, U1 ${PARTNUMBER}

Commit message: Completed v0 board
Parts:
- C5: LCSC C28323 -> (none); LCSC Part (none) -> C52923; PARTNUMBER C1608X7R1C105K -> CL05A105KA5NQNC
- Q1, Q2, Q3, Q4: PARTNUMBER CSD18532Q5B -> CSD18540Q5B
- R1, R2, R4: LCSC C25744 -> C1160
